File: kicad/ProPrj_Neon_2025-07-07.kicad_pcb (KiCad board)
At the start: 2 copper layers, 19.3 x 17.3 mm, 13 parts

Commit message: fix pcb symbols
Parts:
- C1, C3: value (none) -> 100nF
- C2: value (none) -> 100nF; footprint ProPrj_Neon_2025-07-07:C0805 -> ProPrj_Neon_2025-07-07:C0603
- D2: value (none) -> SOD4007-MS
- Q1: value (none) -> BSS123
- R3: value (none) -> 10K
- R4: value (none) -> 100kΩ
- R5: value (none) -> 1Ω
- U2: value (none) -> NE555-TD
- U3, USB1: value (none) -> ~
- U4: value (none) -> BAV99
- U5: value (none) -> 47uH
Connections:
- net $1N1148 renamed Net-(D2-K)
- net $1N1405 renamed Net-(R3-Pad2)
- net $1N1856 renamed Net-(R4-Pad1)
- net $1N1862 renamed Net-(R4-Pad3)
- net $1N2753 renamed Net-(R5-Pad1)
- net $1N996 renamed Net-(D2-A)
- net +5V renamed <NO NET>
- net OUT renamed /OUT
- net TRIG renamed /TRIG
- U2 pad 5: (no net) -> unconnected-(U2-Cont-Pad5)
- U2 pad 7: (no net) -> unconnected-(U2-Disch-Pad7)
- USB1 pad 2: (no net) -> unconnected-(USB1-D--Pad2)
- USB1 pad 3: (no net) -> unconnected-(USB1-D+-Pad3)
Routing:
- net GND: vias 6 -> 0
- net (no net): vias 0 -> 6
